Commit message: Bugfixes

File: phoenixbot_description/urdf/phoenixbot_simon.xacro (robot description, xacro)
@@ -48,8 +48,8 @@
     <joint name="simon_arm_joint" type="revolute">
         <axis xyz="0 1 0"/>
-        <origin xyz="${-10.73 * IN} 0 ${3 * IN}"/>
+        <origin xyz="${-10.73 * IN} 0 ${3 * IN}" rpy="0 ${pi/2} 0"/>
         <parent link="chassis"/>
         <child link="simon_arm"/>
-        <limit lower="0" upper="1.6" effort="20.0" velocity="1.6"/>
+        <limit lower="0" upper="1.57" effort="20.0" velocity="1.6"/>
     </joint>
     <transmission name="simon_arm_transmission">

Commit message: Fixed bugs in simon arm description

File: phoenixbot_description/urdf/phoenixbot_simon.xacro (robot description, xacro)
@@ -51,13 +51,13 @@
         <parent link="chassis"/>
         <child link="simon_arm"/>
-        <limit lower="0" upper="1.57" effort="20.0" velocity="1.6"/>
+        <limit lower="${-pi / 2}" upper="1" effort="20.0" velocity="${pi/2}"/>
     </joint>
     <transmission name="simon_arm_transmission">
         <type>transmission_interface/SimpleTransmission</type>
         <joint name="simon_arm_joint">
-            <hardwareInterface>hardware_interface/VelocityJointInterface</hardwareInterface>
+            <hardwareInterface>hardware_interface/PositionJointInterface</hardwareInterface>
         </joint>
         <actuator name="simon_motor">
-            <hardwareInterface>hardware_interface/VelocityJointInterface</hardwareInterface>
+            <hardwareInterface>hardware_interface/PositionJointInterface</hardwareInterface>
             <mechanicalReduction>1</mechanicalReduction>
         </actuator>

Commit message: Fixed bug in simon arm command

File: phoenixbot_description/urdf/phoenixbot_simon.xacro (robot description, xacro)
@@ -51,5 +51,5 @@
         <parent link="chassis"/>
         <child link="simon_arm"/>
-        <limit lower="${-pi / 2}" upper="1" effort="20.0" velocity="${pi/2}"/>
+        <limit lower="${-pi / 2}" upper="${pi/4}" effort="20.0" velocity="${pi/2}"/>
     </joint>
     <transmission name="simon_arm_transmission">

Commit message: Changed simon arm starting angle

File: phoenixbot_description/urdf/phoenixbot_simon.xacro (robot description, xacro)
@@ -51,5 +51,5 @@
         <parent link="chassis"/>
         <child link="simon_arm"/>
-        <limit lower="${-pi / 2}" upper="${pi/4}" effort="20.0" velocity="${pi/2}"/>
+        <limit lower="${-pi / 2}" upper="${33 * DEG}" effort="20.0" velocity="${pi/2}"/>
     </joint>
     <transmission name="simon_arm_transmission">

File: phoenixbot_description/urdf/util.xacro (robot description, xacro)
@@ -2,4 +2,5 @@
 <robot xmlns:xacro="http://www.ros.org/wiki/xacro" name="phoenixbot">
     <xacro:property name="IN" value="0.0254" />
+    <xacro:property name="DEG" value="${pi/180}" />
     <xacro:property name="LBS" value="0.453592" />
     <xacro:macro name="cylinder_inertia" params="mass radius thickness">
