Commit message: Updated description

File: phoenixbot_description/urdf/phoenixbot.urdf.xacro (robot description, xacro)
@@ -8,5 +8,4 @@
     <xacro:include filename="$(find phoenixbot_description)/urdf/phoenixbot_chassis.xacro" />
     <xacro:include filename="$(find phoenixbot_description)/urdf/phoenixbot_simon.xacro" />
-    <xacro:include filename="$(find phoenixbot_description)/urdf/phoenixbot_pulley.xacro" />
 	<link name="camera"/>
 	<joint name="camera_joint" type="fixed">
@@ -25,5 +24,5 @@
 		<parent link="base_link"/>
 		<child link="laser_link"/>
-        <origin xyz="${10.73 * IN} 0 ${3 * IN}"/>
+        <origin xyz="0.3360 0.3184 0.0883"/>
 	</joint>
 </robot>

File: phoenixbot_description/urdf/phoenixbot_chassis.xacro (robot description, xacro)
@@ -1,13 +1,20 @@
 <?xml version="1.0"?>
 <robot xmlns:xacro="http://www.ros.org/wiki/xacro" name="phoenixbot_chassis">
-    <xacro:macro name="wheel" params="name pos">
-        <link name="${name}">
+    <xacro:macro name="wheel" params="pos side">
+      <link name="${side}_${pos}_wheel">
             <visual>
-                <!--<origin rpy="0 0 ${pi/2}"/>-->
-                <origin rpy="${pi/2} 0 0"/>
+              <xacro:if value="${side == 'right'}">
+                <origin rpy="0 0 ${pi}"/>
+              </xacro:if>
+              <xacro:if value="${pos == 'front' or pos=='back'}">
                 <geometry>
-				<!--<mesh filename = "package://phoenixbot_description/meshes/${pos}.stl" scale="0.01 0.01 0.01"/>-->
-                    <cylinder length="${1 * IN}" radius="${3 * IN}"/>
+                  <mesh filename = "package://phoenixbot_description/meshes/2019/outer_wheel.dae" scale="0.01 0.01 0.01"/>
                 </geometry>
+              </xacro:if>
+              <xacro:if value="${pos == 'center'}">
+                <geometry>
+                  <mesh filename = "package://phoenixbot_description/meshes/2019/center_wheel.dae" scale="0.01 0.01 0.01"/>
+                </geometry>
+              </xacro:if>
             </visual>
             <collision>
@@ -31,17 +38,27 @@
         <parent link="base_link"/>
         <child link="chassis"/>
-        <origin xyz="0 0 ${1 * IN}"/>
+        <origin xyz="0 0 -0.0212"/>
     </joint>
     <joint name = "base_footprint_joint" type="fixed">
-        <parent link="base_link"/>
+        <parent link="chassis"/>
         <child link="base_footprint"/>
         <origin xyz="0 0 ${-3 * IN}"/>
     </joint>
+    <link name="superstructure">
+        <visual>
+            <geometry>
+              <mesh filename = "package://phoenixbot_description/meshes/2019/superstructure.dae" scale="0.01 0.01 0.01"/>
+            </geometry>
+        </visual>
+    </link>
+    <joint name = "superstructure_joint" type="fixed">
+        <parent link="chassis"/>
+        <child link="superstructure"/>
+        <origin xyz="0 0 0.0755"/>
+    </joint>
     <link name="chassis">
         <visual>
-	    <origin rpy="${pi/2} 0 ${pi/2}"/>
             <geometry>
-		<mesh filename = "package://phoenixbot_description/meshes/phoenixbotbody.stl" scale="0.01 0.01 0.01"/>
-                <!--<box size="${28.31 * IN} ${27.50 * IN} ${3.33 * IN}"/>-->
+              <mesh filename = "package://phoenixbot_description/meshes/2019/chassis.dae" scale="0.01 0.01 0.01"/>
             </geometry>
         </visual>
@@ -60,25 +77,25 @@
     </link>
     <!-- Left wheels -->
-    <xacro:wheel name="left_wheel" pos="middle_center"/>
-    <xacro:wheel name="left_fwheel" pos="outerWheel_center"/>
-    <xacro:wheel name="left_rwheel" pos="outerWheel_center"/>
+    <xacro:wheel side="left" pos="center"/>
+    <xacro:wheel side="left" pos="front"/>
+    <xacro:wheel side="left" pos="back"/>
     <joint name="left_wheel_joint" type="continuous">
         <axis xyz="0 1 0"/>
-        <origin xyz="0 ${11.4 * IN} -${0.5 * IN}"/> <!-- 0 ${12.82 *IN} 0 -->
-        <parent link="base_link"/>
-        <child link="left_wheel"/>
+        <origin xyz="0 0.3012 0.0"/>
+        <parent link="chassis"/>
+        <child link="left_center_wheel"/>
     </joint>
-    <joint name="left_fwheel_joint" type="continuous">
+    <joint name="left_front_wheel_joint" type="continuous">
         <axis xyz="0 1 0"/>
-        <origin xyz="${10.73 * IN} ${11.4 * IN} ${0.25 * IN}"/>
-        <parent link="base_link"/>
-        <child link="left_fwheel"/>
+        <origin xyz="0.2725 0.3057 0.0003556"/>
+        <parent link="chassis"/>
+        <child link="left_front_wheel"/>
         <mimic joint="left_wheel_joint"/>
     </joint>
-    <joint name="left_rwheel_joint" type="continuous">
+    <joint name="left_back_wheel_joint" type="continuous">
         <axis xyz="0 1 0"/>
-        <origin xyz="${-10.73 * IN} ${11.4 * IN} ${0.25 * IN}"/>
-        <parent link="base_link"/>
-        <child link="left_rwheel"/>
+        <origin xyz="-0.2725 0.3057 0.0003556"/>
+        <parent link="chassis"/>
+        <child link="left_back_wheel"/>
         <mimic joint="left_wheel_joint"/>
     </joint>
@@ -94,25 +111,25 @@
     </transmission>
     <!-- Right wheels -->
-    <xacro:wheel name="right_wheel" pos="middle_center"/>
-    <xacro:wheel name="right_fwheel" pos="outerWheel_center"/>
-    <xacro:wheel name="right_rwheel" pos="outerWheel_center"/>
+    <xacro:wheel side="right" pos="center"/>
+    <xacro:wheel side="right" pos="front"/>
+    <xacro:wheel side="right" pos="back"/>
     <joint name="right_wheel_joint" type="continuous">
         <axis xyz="0 1 0"/>
-        <origin xyz="0 ${-12.82 * IN} 0"/>
-        <parent link="base_link"/>
-        <child link="right_wheel"/>
+        <origin xyz="0 -0.3012 0.0"/>
+        <parent link="chassis"/>
+        <child link="right_center_wheel"/>
     </joint>
-    <joint name="right_fwheel_joint" type="continuous">
+    <joint name="right_front_wheel_joint" type="continuous">
         <axis xyz="0 1 0"/>
-        <origin xyz="${10.73 * IN} ${-12.82 * IN} ${0.25 * IN}"/>
-        <parent link="base_link"/>
-        <child link="right_fwheel"/>
+        <origin xyz="0.2725 -0.3057 0.0003556"/>
+        <parent link="chassis"/>
+        <child link="right_front_wheel"/>
         <mimic joint="right_wheel_joint"/>
     </joint>
-    <joint name="right_rwheel_joint" type="continuous">
+    <joint name="right_back_wheel_joint" type="continuous">
         <axis xyz="0 1 0"/>
-        <origin xyz="${-10.73 * IN} ${-12.82 * IN} ${0.25 * IN}"/>
-        <parent link="base_link"/>
-        <child link="right_rwheel"/>
+        <origin xyz="-0.2725 -0.3057 0.0003556"/>
+        <parent link="chassis"/>
+        <child link="right_back_wheel"/>
         <mimic joint="right_wheel_joint"/>
     </joint>

File: phoenixbot_description/urdf/phoenixbot_simon.xacro (robot description, xacro)
@@ -5,48 +5,44 @@
             <origin rpy="0 0 0"/>
             <geometry>
-                <mesh filename="package://phoenixbot_description/meshes/simonArm.stl"/>
+              <mesh filename="package://phoenixbot_description/meshes/2019/simon_arm.dae" scale="0.01 0.01 0.01"/>
             </geometry>
         </visual>
-        <collision>
-            <origin xyz="${-14 * IN} 0 0"/>
+        <xacro:trivial_inertia/>
+    </link>
+    <link name="left_paddle">
+        <visual>
+            <origin rpy="0 0 0"/>
             <geometry>
-                <box size="${29.5 * IN} ${24 * IN} ${3 * IN}"/>
+              <mesh filename="package://phoenixbot_description/meshes/2019/left_paddle.dae" scale="0.01 0.01 0.01"/>
             </geometry>
-        </collision>
-        <inertial>
-            <mass value="${4 * LBS}"/>
-            <inertia ixx="${1/12*15*LBS*((3.33*IN)**2+(28.31*IN)**2)}"
-                iyy="${1/12*15*LBS*((27.50*IN)**2+(28.31*IN)**2)}"
-                izz="${1/12*15*LBS*((27.50*IN)**2+(3.33*IN)**2)}"
-            ixy="0" ixz="0" iyz="0"/>
-        </inertial>
+        </visual>
+        <xacro:trivial_inertia/>
     </link>
-    <link name="solenoid1"/>
-    <link name="solenoid2"/>
-    <link name="solenoid3"/>
-    <link name="solenoid4"/>
-    <joint name="solenoid1_joint" type="fixed">
+    <link name="right_paddle">
+        <visual>
+            <origin rpy="0 0 0"/>
+            <geometry>
+              <mesh filename="package://phoenixbot_description/meshes/2019/right_paddle.dae" scale="0.01 0.01 0.01"/>
+            </geometry>
+        </visual>
+        <xacro:trivial_inertia/>
+    </link>
+    <joint name="left_paddle_joint" type="revolute">
+        <axis xyz="0 1 0"/>
+        <origin xyz="-0.3047 0.14 0.0539" rpy="0 0 0"/>
         <parent link="simon_arm"/>
-        <child link="solenoid1"/>
-        <origin xyz="${-28 * IN} ${-5 * IN} 0"/>
+        <child link="left_paddle"/>
+        <limit lower="${-45 * DEG}" upper="${45 * DEG}" effort="20.0" velocity="${pi/2}"/>
     </joint>
-    <joint name="solenoid2_joint" type="fixed">
+    <joint name="right_paddle_joint" type="revolute">
+        <axis xyz="0 1 0"/>
+        <origin xyz="-0.3047 -0.14 0.0539" rpy="0 0 0"/>
         <parent link="simon_arm"/>
-        <child link="solenoid2"/>
-        <origin xyz="${-28 * IN} ${5 * IN} 0"/>
-    </joint>
-    <joint name="solenoid3_joint" type="fixed">
-        <parent link="simon_arm"/>
-        <child link="solenoid3"/>
-        <origin xyz="${-18 * IN} ${5 * IN} 0"/>
-    </joint>
-    <joint name="solenoid4_joint" type="fixed">
-        <parent link="simon_arm"/>
-        <child link="solenoid4"/>
-        <origin xyz="${-18 * IN} ${-5 * IN} 0"/>
+        <child link="right_paddle"/>
+        <limit lower="${-45 * DEG}" upper="${45 * DEG}" effort="20.0" velocity="${pi/2}"/>
     </joint>
     <joint name="simon_arm_joint" type="revolute">
         <axis xyz="0 1 0"/>
-        <origin xyz="${-10.73 * IN} 0 ${3 * IN}" rpy="0 ${pi/2} 0"/>
+        <origin xyz="-0.3105 0 0.1073" rpy="0 ${pi/2} 0"/>
         <parent link="chassis"/>
         <child link="simon_arm"/>
@@ -63,3 +59,23 @@
         </actuator>
     </transmission>
+    <transmission name="left_paddle_transmission">
+        <type>transmission_interface/SimpleTransmission</type>
+        <joint name="left_paddle_joint">
+            <hardwareInterface>hardware_interface/PositionJointInterface</hardwareInterface>
+        </joint>
+        <actuator name="left_paddle_servo">
+            <hardwareInterface>hardware_interface/PositionJointInterface</hardwareInterface>
+            <mechanicalReduction>1</mechanicalReduction>
+        </actuator>
+    </transmission>
+    <transmission name="right_paddle_transmission">
+        <type>transmission_interface/SimpleTransmission</type>
+        <joint name="right_paddle_joint">
+            <hardwareInterface>hardware_interface/PositionJointInterface</hardwareInterface>
+        </joint>
+        <actuator name="right_paddle_servo">
+            <hardwareInterface>hardware_interface/PositionJointInterface</hardwareInterface>
+            <mechanicalReduction>1</mechanicalReduction>
+        </actuator>
+    </transmission>
 </robot>

File: phoenixbot_description/urdf/util.xacro (robot description, xacro)
@@ -11,3 +11,10 @@
         </inertial>
     </xacro:macro>
+    <xacro:macro name="trivial_inertia">
+        <xacro:property name="INERTIA" value="0.01"/>
+        <inertial>
+            <mass value="0.01"/>
+            <inertia ixx="${INERTIA}" iyy="${INERTIA}" izz="${INERTIA}" ixy="0" ixz="0" iyz="0"/>
+        </inertial>
+    </xacro:macro>
 </robot>
