Commit message: Added nav stack and fixed simulation

File: phoenixbot_description/urdf/phoenixbot_chassis.xacro (robot description, xacro)
@@ -19,8 +19,14 @@
 	</xacro:macro>
     <link name="base_link"/>
+    <link name="base_footprint"/>
     <joint name = "base_link_joint" type="fixed">
         <parent link="base_link"/>
         <child link="chassis"/>
         <origin xyz="0 0 ${1 * IN}"/>
+    </joint>
+    <joint name = "base_footprint_joint" type="fixed">
+        <parent link="base_link"/>
+        <child link="base_footprint"/>
+        <origin xyz="0 0 0"/>
     </joint>
     <link name="chassis">

Commit message: Updated chassis and wheels. Wheels are not centered

File: phoenixbot_description/urdf/phoenixbot_chassis.xacro (robot description, xacro)
@@ -1,10 +1,11 @@
 <?xml version="1.0"?>
 <robot xmlns:xacro="http://www.ros.org/wiki/xacro" name="phoenixbot_chassis">
-    <xacro:macro name="wheel" params="name">
+    <xacro:macro name="wheel" params="name pos">
         <link name="${name}">
             <visual>
-                <origin rpy="${pi/2} 0 0"/>
+                <origin rpy="0 0 ${pi/2}"/>
                 <geometry>
-                    <cylinder length="${1 * IN}" radius="${2 * IN}"/>
+		    <mesh filename = "package://phoenixbot_description/meshes/${pos}.stl" scale="0.01 0.01 0.01"/>
+                    <!--<cylinder length="${1 * IN}" radius="${2 * IN}"/>-->
                 </geometry>
             </visual>
@@ -32,6 +33,8 @@
     <link name="chassis">
         <visual>
+	    <origin rpy="${pi/2} 0 ${pi/2}"/>
             <geometry>
-                <box size="${28.31 * IN} ${27.50 * IN} ${3.33 * IN}"/>
+		<mesh filename = "package://phoenixbot_description/meshes/phoenixbotbody.stl" scale="0.01 0.01 0.01"/>
+                <!--<box size="${28.31 * IN} ${27.50 * IN} ${3.33 * IN}"/>-->
             </geometry>
         </visual>
@@ -41,5 +44,5 @@
             </geometry>
         </collision>
-        <inertial>
+        <inertial>pi
             <mass value="${15 * LBS}"/>
             <inertia ixx="${1/12*15*LBS*((3.33*IN)**2+(28.31*IN)**2)}"
@@ -50,7 +53,7 @@
     </link>
     <!-- Left wheels -->
-    <xacro:wheel name="left_wheel"/>
-    <xacro:wheel name="left_fwheel"/>
-    <xacro:wheel name="left_rwheel"/>
+    <xacro:wheel name="left_wheel" pos="middle2"/>
+    <xacro:wheel name="left_fwheel" pos="top2"/>
+    <xacro:wheel name="left_rwheel" pos="bottom2"/>
     <joint name="left_wheel_joint" type="continuous">
         <axis xyz="0 1 0"/>
@@ -84,7 +87,7 @@
     </transmission>
     <!-- Right wheels -->
-    <xacro:wheel name="right_wheel"/>
-    <xacro:wheel name="right_fwheel"/>
-    <xacro:wheel name="right_rwheel"/>
+    <xacro:wheel name="right_wheel" pos="middle1"/>
+    <xacro:wheel name="right_fwheel" pos="top1"/>
+    <xacro:wheel name="right_rwheel" pos="bottom1"/>
     <joint name="right_wheel_joint" type="continuous">
         <axis xyz="0 1 0"/>

Commit message: Add mesh to chassis and wheel. The wheel mesh is wrong.

File: phoenixbot_description/urdf/phoenixbot_chassis.xacro (robot description, xacro)
@@ -53,10 +53,10 @@
     </link>
     <!-- Left wheels -->
-    <xacro:wheel name="left_wheel" pos="middle2"/>
-    <xacro:wheel name="left_fwheel" pos="top2"/>
-    <xacro:wheel name="left_rwheel" pos="bottom2"/>
+    <xacro:wheel name="left_wheel" pos="middle_center"/>
+    <xacro:wheel name="left_fwheel" pos="outerWheel_center"/>
+    <xacro:wheel name="left_rwheel" pos="outerWheel_center"/>
     <joint name="left_wheel_joint" type="continuous">
         <axis xyz="0 1 0"/>
-        <origin xyz="0 ${12.82 * IN} 0"/>
+        <origin xyz="0 ${11.4 * IN} -${0.5 * IN}"/> <!-- 0 ${12.82 *IN} 0 -->
         <parent link="base_link"/>
         <child link="left_wheel"/>
@@ -87,7 +87,7 @@
     </transmission>
     <!-- Right wheels -->
-    <xacro:wheel name="right_wheel" pos="middle1"/>
-    <xacro:wheel name="right_fwheel" pos="top1"/>
-    <xacro:wheel name="right_rwheel" pos="bottom1"/>
+    <xacro:wheel name="right_wheel" pos="middle_center"/>
+    <xacro:wheel name="right_fwheel" pos="outerWheel_center"/>
+    <xacro:wheel name="right_rwheel" pos="outerWheel_center"/>
     <joint name="right_wheel_joint" type="continuous">
         <axis xyz="0 1 0"/>

Commit message: Added IMU link to chassis

File: phoenixbot_description/urdf/phoenixbot_chassis.xacro (robot description, xacro)
@@ -20,4 +20,10 @@
         </link>
 	</xacro:macro>
+  <link name="imu_link"/>
+  <joint name = "imu_joint" type="fixed">
+      <parent link="base_link"/>
+      <child link="imu_link"/>
+      <origin xyz="${-1.5 * IN} ${-2 * IN} 0"/>
+  </joint>
     <link name="base_link"/>
     <link name="base_footprint"/>

Commit message: Updated gazebo simulation parameters

File: phoenixbot_description/urdf/phoenixbot_chassis.xacro (robot description, xacro)
@@ -64,6 +64,7 @@
         </visual>
         <collision>
+            <origin xyz="0 0 0.03"/>
             <geometry>
-                <box size="${28.31 * IN} ${27.50 * IN} ${3.33 * IN}"/>
+                <box size="0.7108 0.7190 0.0866"/>
             </geometry>
         </collision>

File: phoenixbot_description/urdf/phoenixbot_simon.xacro (robot description, xacro)
@@ -47,5 +47,5 @@
         <parent link="chassis"/>
         <child link="simon_arm"/>
-        <limit lower="${-pi / 2}" upper="${33 * DEG}" effort="20.0" velocity="${pi/2}"/>
+        <limit lower="${-pi / 2}" upper="${33 * DEG}" effort="20.0" velocity="${pi/10}"/>
     </joint>
     <transmission name="simon_arm_transmission">
